File: din_meter_atm90e26.kicad_pcb (KiCad board)
At the start: 2 copper layers, 29 x 31.2 mm, 48 parts, among them J1 USEL, J2 MMD1, J3 MMD0, J4 CONN_02X18, J5 CONN_01X10, J6 USEL, J7 MMD1, J8 MMD0, M1 ATM90E26_ATM90E26, M2 ATM90E26_ATM90E26, Y1 Crystal_Small, Y2 Crystal_Small

Commit message: Add labels to PCI-X
Connections:
- J4 pad A1: Net-(J4-PadA1) -> 3V3_ISO
- J4 pad A12: Net-(J4-PadA12) -> GND_CPU
- J4 pad A16: Net-(J4-PadA16) -> 3V3_CPU
- J4 pad A2: Net-(J4-PadA2) -> VP_0
- J4 pad A4: Net-(J4-PadA4) -> VP_1
- J4 pad A8: Net-(J4-PadA8) -> GNDREF
- J4 pad B3: Net-(J4-PadB3) -> I1N_1_IN
- J4 pad B4: Net-(J4-PadB4) -> I1P_1_IN
- J4 pad B5: Net-(J4-PadB5) -> I1N_0_IN
- J4 pad B6: Net-(J4-PadB6) -> I1P_0_IN
- J5 pad 10: GND_ISO -> GND_CPU
- J5 pad 2: 3V3_IN -> 3V3_ISO
- J5 pad 9: 3V3_ISO -> 3V3_CPU

Commit message: v0.1 prepped for fab
Parts:
- added CF1_0: CF1_0, Measurement_Points:Measurement_Point_Round-SMD-Pad_Small, B.Cu at (150.4, 68.5)
- added CF1_1: CF1_1, Measurement_Points:Measurement_Point_Round-SMD-Pad_Small, B.Cu at (141.6, 73.5)
- added CF2_0: CF2_0, Measurement_Points:Measurement_Point_Round-SMD-Pad_Small, B.Cu at (150.4, 71.0)
- added CF2_1: CF2_1, Measurement_Points:Measurement_Point_Round-SMD-Pad_Small, B.Cu at (141.6, 71.0)
- added IRQ_0: IRQ_0, Measurement_Points:Measurement_Point_Round-SMD-Pad_Small, B.Cu at (150.4, 73.5)
- added IRQ_1: IRQ_1, Measurement_Points:Measurement_Point_Round-SMD-Pad_Small, B.Cu at (141.6, 68.5)
- added L1: GND_SUP, Inductors_SMD:L_0402, F.Cu at (142.5, 80.7)
- added L2: 3V3_SUP, Inductors_SMD:L_0402, F.Cu at (136.0, 80.8)
- added WARN_0: WARN_0, Measurement_Points:Measurement_Point_Round-SMD-Pad_Small, B.Cu at (150.4, 65.9)
- added WARN_1: WARN_1, Measurement_Points:Measurement_Point_Round-SMD-Pad_Small, B.Cu at (141.6, 76.1)
- added ZX_0: ZX_0, Measurement_Points:Measurement_Point_Round-SMD-Pad_Small, B.Cu at (150.4, 76.1)
- added ZX_1: ZX_1, Measurement_Points:Measurement_Point_Round-SMD-Pad_Small, B.Cu at (141.6, 65.9)
- C13, C14, C6, C7: value C_Small -> 20p
- moved G1 1.91 mm to (145.7, 75.8)
- turned LOGO1 to 270 degrees
Connections:
- C1 pad 1: Net-(C1-Pad1) -> +3V3
- C10 pad 1: Net-(C10-Pad1) -> +3V3
- C10 pad 2: GNDREF -> GNDD
- C11 pad 2: GNDREF -> GNDD
- C12 pad 2: GNDREF -> GNDD
- C15 pad 1: GNDREF -> GNDD
- C16 pad 1: GNDREF -> GNDD
- C17 pad 1: GNDREF -> GNDD
- C18 pad 1: GNDREF -> GNDD
- C19 pad 1: GNDREF -> GNDD
- C2 pad 2: Net-(C1-Pad1) -> +3V3
- C20 pad 1: GNDREF -> GNDD
- C21 pad 1: GNDREF -> GNDD
- C22 pad 1: GNDREF -> GNDD
- C23 pad 1: GNDREF -> GNDD
- C24 pad 1: GNDREF -> GNDD
- C3 pad 1: Net-(C3-Pad1) -> +3V3
- C3 pad 2: GNDREF -> GNDD
- C4 pad 2: GNDREF -> GNDD
- C5 pad 2: GNDREF -> GNDD
- C8 pad 1: Net-(C8-Pad1) -> +3V3
- C9 pad 2: Net-(C8-Pad1) -> +3V3
- J4 pad A8: GNDREF -> GND_ISO
- J4 pad B12: Net-(J4-PadB12) -> I2P_0_IN
- J4 pad B14: Net-(J4-PadB14) -> I2N_0_IN
- J4 pad B16: Net-(J4-PadB16) -> I2P_1_IN
- J4 pad B18: Net-(J4-PadB18) -> I2N_1_IN
- J5 pad 1: GNDREF -> 3V3_CPU
- J5 pad 10: GND_CPU -> 3V3_ISO
- J5 pad 2: 3V3_ISO -> GND_CPU
- J5 pad 3: SI/RX -> Net-(J5-Pad3)
- J5 pad 4: SO/TX -> CS_0
- J5 pad 6: CS_0 -> SO/TX
- J5 pad 7: CS_1 -> SI/RX
- J5 pad 8: Net-(J5-Pad8) -> CS_1
- J5 pad 9: 3V3_CPU -> GND_ISO
- M1 pad 14: GNDREF -> GNDD
- M1 pad 3: Net-(C1-Pad1) -> +3V3
- M1 pad 4: Net-(C1-Pad1) -> +3V3
- M1 pad 5: Net-(C3-Pad1) -> +3V3
- M1 pad 6: GNDREF -> GNDD
- M2 pad 14: GNDREF -> GNDD
- M2 pad 3: Net-(C8-Pad1) -> +3V3
- M2 pad 4: Net-(C8-Pad1) -> +3V3
- M2 pad 5: Net-(C10-Pad1) -> +3V3
- M2 pad 6: GNDREF -> GNDD
- R1 pad 2: GNDREF -> GNDD
- R2 pad 2: GNDREF -> GNDD
Routing:
- net GNDD: track 0.00 -> 165.3 mm, vias 0 -> 4
- net +3V3: track 0.00 -> 83.9 mm, vias 0 -> 6
- net I2P_1_IN: track 0.00 -> 55.7 mm, vias 0 -> 2
- net I2N_0_IN: track 0.00 -> 44.4 mm, vias 0 -> 4
- net I2N_1_IN: track 0.00 -> 37.2 mm, vias 0 -> 2
- net VP_0: track 0.00 -> 31.0 mm, vias 0 -> 1
- net GND_CPU: track 0.00 -> 30.6 mm
- net GND_ISO: track 0.00 -> 30.2 mm, vias 0 -> 2
- net 3V3_CPU: track 0.00 -> 27.5 mm
- net 3V3_ISO: track 0.00 -> 27.3 mm, vias 0 -> 1
- net I2P_0_IN: track 0.00 -> 25.1 mm, vias 0 -> 4
- net SCLK: track 0.00 -> 20.8 mm
- net SI/RX: track 0.00 -> 20.4 mm, vias 0 -> 2
- net SO/TX: track 0.00 -> 19.7 mm, vias 0 -> 2
- net VP_1: track 0.00 -> 19.0 mm, vias 0 -> 1
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Other:
- net class Default: clearance 0.2 -> 0.15; trace_width 0.25 -> 0.15; via_dia 0.8 -> 0.6; via_drill 0.4 -> 0.3
- net class Power_CPU added: clearance 0.4, trace_width 0.4, via_dia 0.6, via_drill 0.3
- net class Power_ISO added: clearance 0.2, trace_width 0.3, via_dia 0.6, via_drill 0.3
- rule trace_clearance: 0.2 -> 0.15
- rule trace_min: 0.2 -> 0.15
- rule via_min_size: 0.4 -> 0.6
- board text added: "3V3_C"
- board text added: "3V3_I"
- board text added: "CLK"
- board text added: "CS_0"
- board text added: "CS_1"
- board text added: "Dual ATM90E26 v0.1 16/10/2017"
- board text added: "GND_C"
- board text added: "GND_I"
- board text added: "SI"
- board text added: "SO"
