File: din_meter_atm90e26.sch (KiCad schematic (older format))
At the start: 61 parts, among them J1 USEL, J2 MMD1, J3 MMD0, J4 CONN_02X18, J5 CONN_01X10, J6 USEL, J7 MMD1, J8 MMD0, M1 ATM90E26_ATM90E26, M2 ATM90E26_ATM90E26, Y1 Crystal_Small, Y2 Crystal_Small

Commit message: Open soldermask on gold fingers and bump version
Parts:
- Y1: manf# 5XFA08192123TF80Q3 -> AA-8.192MAGE-T
Changed lines of the file:
@@
 F 2 "Crystals:Crystal_SMD_5032-2pin_5.0x3.2mm" H 900 1500 50  0001 C CNN
 F 3 "" H 900 1500 50  0001 C CNN
-F 4 "5XFA08192123TF80Q3" H 900 1500 60  0001 C CNN "manf#"
+F 4 "AA-8.192MAGE-T" H 900 1500 60  0001 C CNN "manf#"
 	1    900  1500
 	1    0    0    -1
